Commit message: increase control frequency add gravity compensation

File: hand_driver/allegro_hand_description/allegro_hand_description_right.urdf (robot description, URDF)
Before this commit: robot allegro_hand_right, 22 links, 21 joints
Links:
- added link world
Joints:
- added joint world_joint: type fixed, parent world, child hand_root, origin xyz=0 0 0 rpy=0 1.5708 0

Commit message: add kuka driver

File: hand_driver/allegro_hand_description/allegro_hand_description_right.urdf (robot description, URDF)
Before this commit: robot allegro_hand_right, 23 links, 22 joints
Links:
- link palm_link: geometry collision box size=0.0408 0.1130 0.095; visual mesh filename=package://allegro_hand_description/meshes/base_link_mod.stl
