Commit message: add left hand

File: hand_driver/allegro_hand_description/allegro_hand_description_left.urdf (robot description, URDF)
Before this commit: robot allegro_hand_left, 21 links, 20 joints
Links:
- added link hand_root
- added link world
Joints:
- added joint root: type fixed, parent hand_root, child palm_link, origin xyz=0 0 0 rpy=0 0 0
- added joint world_joint: type fixed, parent world, child hand_root, origin xyz=0 0 0 rpy=0 1.5708 0
